Commit message: update

File: description/alpha/urdf/alpha_5.urdf.xacro (robot description, xacro)
@@ -178,4 +178,37 @@
             <origin xyz="0 0 0" rpy="0 0 0"/>
         </xacro:alpha_standard_jaws>
+        <link name="${name}_payload">
+        <!-- optional inertia if you want it in dynamics -->
+        <inertial>
+            <mass value="2.0"/>
+            <inertia
+            ixx="1e-4" ixy="0.0" ixz="0.0"
+            iyy="1e-4" iyz="0.0"
+            izz="1e-4"/>
+        </inertial>
+        <visual>
+            <!-- raise the box half its height so it sits flush on the tip -->
+            <origin xyz="0 0 0.025" rpy="0 0 0"/>
+            <geometry>
+            <box size="0.05 0.05 0.05"/>
+            </geometry>
+            <material name="payload_blue">
+            <color rgba="0 0 1 1"/>
+            </material>
+        </visual>
+        <collision>
+            <origin xyz="0 0 0.025" rpy="0 0 0"/>
+            <geometry>
+            <box size="0.05 0.05 0.05"/>
+            </geometry>
+        </collision>
+        </link>
+        <joint name="${name}_payload_joint" type="fixed">
+        <!-- swap this parent to whichever link is your true tip -->
+        <parent link="${name}_jaws_base_link"/>
+        <child  link="${name}_payload"/>
+        <!-- adjust this if your tip is elsewhere or rotated differently -->
+        <origin xyz="0 0 0.04" rpy="0 0 0"/>
+        </joint>
     </xacro:macro>
 </robot>

Commit message: endeffector model added

File: description/alpha/urdf/alpha_5.urdf.xacro (robot description, xacro)
@@ -178,6 +178,5 @@
             <origin xyz="0 0 0" rpy="0 0 0"/>
         </xacro:alpha_standard_jaws>
-        <link name="${name}_payload">
-        <!-- optional inertia if you want it in dynamics -->
+        <!-- <link name="${name}_payload">
         <inertial>
             <mass value="2.0"/>
@@ -188,5 +187,4 @@
         </inertial>
         <visual>
-            <!-- raise the box half its height so it sits flush on the tip -->
             <origin xyz="0 0 0.025" rpy="0 0 0"/>
             <geometry>
@@ -203,12 +201,10 @@
             </geometry>
         </collision>
-        </link>
-        <joint name="${name}_payload_joint" type="fixed">
-        <!-- swap this parent to whichever link is your true tip -->
+        </link> -->
+        <!-- <joint name="${name}_payload_joint" type="fixed">
         <parent link="${name}_jaws_base_link"/>
         <child  link="${name}_payload"/>
-        <!-- adjust this if your tip is elsewhere or rotated differently -->
         <origin xyz="0 0 0.04" rpy="0 0 0"/>
-        </joint>
+        </joint> -->
     </xacro:macro>
 </robot>
