Commit message: update update meshes

File: description/xacro/robot_system_multi_interface.urdf.xacro (robot description, xacro)
@@ -10,4 +10,6 @@
   <xacro:arg name="description_package" default="ros2_control_blue_reach_5"/>
   <xacro:arg name="use_optitrack" default="false"/>
+  <!-- <xacro:arg name="robot_name" default="bruce"/> -->
+  <xacro:arg name="robot_name" default="dory"/>
   <!-- Properties -->
   <xacro:property name="description_package" value="$(arg description_package)"/>
@@ -19,8 +21,9 @@
   <xacro:property name="use_pwm" value="$(arg use_pwm)"/>
   <xacro:property name="use_optitrack" value="$(arg use_optitrack)"/>
+  <xacro:property name="robot_name" value="$(arg robot_name)"/>
   <!-- Define constants -->
   <xacro:property name="d_min" value="1.0"/>
   <!-- Imports -->
-  <xacro:include filename="$(find ros2_control_blue_reach_5)/xacro/world.xacro"/>
+  <xacro:include filename="$(find ${description_package})/xacro/world.xacro"/>
   <xacro:include filename="$(find ${description_package})/xacro/urdf.xacro"/>
   <!-- Import RRBot ros2_control description -->
@@ -44,4 +47,5 @@
       <!-- Instantiate the robot -->
       <xacro:bluerov2_heavy_alpha_urdf
+        robot_name="${robot_name}"
         prefix="${prefix}"
         x="${x_pos}"
@@ -77,4 +81,5 @@
     <!-- Instantiate the real robot -->
     <xacro:bluerov2_heavy_alpha_urdf
+      robot_name="${robot_name}"
       prefix="${prefix}"
       x="0.0"

File: description/xacro/urdf.xacro (robot description, xacro)
@@ -1,5 +1,5 @@
 <?xml version="1.0"?>
 <robot xmlns:xacro="http://ros.org/wiki/xacro">
-  <xacro:macro name="bluerov2_heavy_alpha_urdf" params="prefix x:=0.0 y:=0.0 z:=2.0 rot_r:=0.0 rot_p:=0.0 rot_y:=0.0">
+  <xacro:macro name="bluerov2_heavy_alpha_urdf" params="robot_name prefix x:=0.0 y:=0.0 z:=2.0 rot_r:=0.0 rot_p:=0.0 rot_y:=0.0">
     <link name="${prefix}manipulator_mount_link">
       <visual>
@@ -74,5 +74,6 @@
     <!-- Imports -->
     <xacro:include filename="$(find ros2_control_blue_reach_5)/alpha/urdf/alpha_5.urdf.xacro" />
-    <xacro:include filename="$(find ros2_control_blue_reach_5)/blue/xacro/bluerov2_heavy_reach/urdf.xacro" />
+    <xacro:include filename="$(find ros2_control_blue_reach_5)/blue/xacro/bluerov2_heavy_reach/${robot_name}_urdf.xacro" />
+    <xacro:include filename="$(find ros2_control_blue_reach_5)/blue/xacro/bluerov2_heavy_reach/${robot_name}_urdf.xacro" />
     <!-- Instantiate the Alpha -->
     <xacro:alpha_5 parent="${prefix}manipulator_mount_link" name="${prefix}">
