Commit message: optitrack mocap integration:

File: description/ros2_control/vehicle_system_multi_interface.ros2_control.xacro (robot description, xacro)
@@ -1,5 +1,5 @@
 <?xml version="1.0"?>
 <robot xmlns:xacro="http://www.ros.org/wiki/xacro">
-  <xacro:macro name="vehicle_system_multi_interface" params="name prefix serial_port state_update_frequency use_hardware frame_id child_frame_id map_frame_id max_set_param_attempts">
+  <xacro:macro name="vehicle_system_multi_interface" params="name prefix serial_port state_update_frequency use_hardware world_frame_id body_frame_id map_frame_id mocap_mast_height use_optitrack">
     <ros2_control name="${name}" type="system">
       <hardware>
@@ -7,15 +7,18 @@
           <plugin>ros2_control_blue_reach_5/BlueRovSystemMultiInterfaceHardware</plugin>
           <param name="prefix">${prefix}</param>
-          <param name="frame_id">${frame_id}</param>
-          <param name="child_frame_id">${child_frame_id}</param>
+          <param name="world_frame_id">${world_frame_id}</param>
+          <param name="body_frame_id">${body_frame_id}</param>
           <param name="map_frame_id">${map_frame_id}</param>
-          <param name="max_set_param_attempts">${max_set_param_attempts}</param>
+          <param name="mocap_mast_height">${mocap_mast_height}</param>
+          <param name="use_optitrack">${use_optitrack}</param>
         </xacro:if>
         <xacro:unless value="${use_hardware}">
           <plugin>ros2_control_blue_reach_5/SimVehicleSystemMultiInterfaceHardware</plugin>
           <param name="prefix">${prefix}</param>
-          <param name="frame_id">${frame_id}</param>
-          <param name="child_frame_id">${child_frame_id}</param>
+          <param name="world_frame_id">${world_frame_id}</param>
+          <param name="body_frame_id">${body_frame_id}</param>
           <param name="map_frame_id">${map_frame_id}</param>
+          <param name="mocap_mast_height">${mocap_mast_height}</param>
+          <param name="use_optitrack">${use_optitrack}</param>
         </xacro:unless>
       </hardware>
@@ -211,4 +214,14 @@
         <state_interface name="dvl_speed_y"/>
         <state_interface name="dvl_speed_z"/>
+        <state_interface name="mocap_x"/>
+        <state_interface name="mocap_y"/>
+        <state_interface name="mocap_z"/>
+        <state_interface name="mocap_roll"/>
+        <state_interface name="mocap_pitch"/>
+        <state_interface name="mocap_yaw"/>
+        <state_interface name="mocap_orientation_w"/>
+        <state_interface name="mocap_orientation_x"/>
+        <state_interface name="mocap_orientation_y"/>
+        <state_interface name="mocap_orientation_z"/>
       </gpio>
     </ros2_control>

File: description/xacro/robot_system_multi_interface.urdf.xacro (robot description, xacro)
@@ -8,4 +8,5 @@
   <xacro:arg name="state_update_frequency" default="250"/>
   <xacro:arg name="description_package" default="ros2_control_blue_reach_5"/>
+  <xacro:arg name="use_optitrack" default="false"/>
   <!-- Properties -->
   <xacro:property name="description_package" value="$(arg description_package)"/>
@@ -15,4 +16,5 @@
   <xacro:property name="use_manipulator_hardware" value="$(arg use_manipulator_hardware)"/>
   <xacro:property name="use_vehicle_hardware" value="$(arg use_vehicle_hardware)"/>
+  <xacro:property name="use_optitrack" value="$(arg use_optitrack)"/>
   <!-- Define constants -->
   <xacro:property name="d_min" value="1.0"/>
@@ -59,8 +61,9 @@
       state_update_frequency="${state_update_frequency}"
       use_hardware="false"
-      frame_id="base_link"
-      child_frame_id="${prefix}base_link"
+      world_frame_id="base_link"
+      body_frame_id="${prefix}base_link"
       map_frame_id="${prefix}map"
-      max_set_param_attempts="5"/>
+      mocap_mast_height="0.5"
+      use_optitrack="${use_optitrack}"/>
       <!-- Recursively call the macro for the next robot -->
       <xacro:instantiate_robots index="${index + 1}" count="${count}"/>
@@ -92,8 +95,9 @@
       state_update_frequency="${state_update_frequency}"
       use_hardware="${use_vehicle_hardware}"
-      frame_id="base_link"
-      child_frame_id="${prefix}base_link"
+      world_frame_id="base_link"
+      body_frame_id="${prefix}base_link"
       map_frame_id="${prefix}map"
-      max_set_param_attempts="5"/>
+      mocap_mast_height="0.5"
+      use_optitrack="${use_optitrack}"/>
   </xacro:if>
 </robot>

Commit message: remove optitrack support

File: description/ros2_control/vehicle_system_multi_interface.ros2_control.xacro (robot description, xacro)
@@ -1,5 +1,5 @@
 <?xml version="1.0"?>
 <robot xmlns:xacro="http://www.ros.org/wiki/xacro">
-  <xacro:macro name="vehicle_system_multi_interface" params="name prefix serial_port state_update_frequency use_hardware world_frame_id body_frame_id map_frame_id mocap_mast_height use_optitrack">
+  <xacro:macro name="vehicle_system_multi_interface" params="name prefix serial_port state_update_frequency use_hardware world_frame_id body_frame_id map_frame_id">
     <ros2_control name="${name}" type="system">
       <hardware>
@@ -10,6 +10,4 @@
           <param name="body_frame_id">${body_frame_id}</param>
           <param name="map_frame_id">${map_frame_id}</param>
-          <param name="mocap_mast_height">${mocap_mast_height}</param>
-          <param name="use_optitrack">${use_optitrack}</param>
         </xacro:if>
         <xacro:unless value="${use_hardware}">
@@ -19,6 +17,4 @@
           <param name="body_frame_id">${body_frame_id}</param>
           <param name="map_frame_id">${map_frame_id}</param>
-          <param name="mocap_mast_height">${mocap_mast_height}</param>
-          <param name="use_optitrack">${use_optitrack}</param>
         </xacro:unless>
       </hardware>
@@ -214,14 +210,4 @@
         <state_interface name="dvl_speed_y"/>
         <state_interface name="dvl_speed_z"/>
-        <state_interface name="gt_x"/>
-        <state_interface name="gt_y"/>
-        <state_interface name="gt_z"/>
-        <state_interface name="gt_roll"/>
-        <state_interface name="gt_pitch"/>
-        <state_interface name="gt_yaw"/>
-        <state_interface name="gt_orientation_w"/>
-        <state_interface name="gt_orientation_x"/>
-        <state_interface name="gt_orientation_y"/>
-        <state_interface name="gt_orientation_z"/>
       </gpio>
     </ros2_control>

File: description/xacro/robot_system_multi_interface.urdf.xacro (robot description, xacro)
@@ -63,7 +63,5 @@
       world_frame_id="base_link"
       body_frame_id="${prefix}base_link"
-      map_frame_id="${prefix}map"
-      mocap_mast_height="0.0"
-      use_optitrack="${use_optitrack}"/>
+      map_frame_id="${prefix}map"/>
       <!-- Recursively call the macro for the next robot -->
       <xacro:instantiate_robots index="${index + 1}" count="${count}"/>
@@ -97,7 +95,5 @@
       world_frame_id="base_link"
       body_frame_id="${prefix}base_link"
-      map_frame_id="${prefix}map"
-      mocap_mast_height="0.0"
-      use_optitrack="${use_optitrack}"/>
+      map_frame_id="${prefix}map"/>
   </xacro:if>
 </robot>

Commit message: added direct thruster control

File: description/ros2_control/vehicle_system_multi_interface.ros2_control.xacro (robot description, xacro)
@@ -1,5 +1,5 @@
 <?xml version="1.0"?>
 <robot xmlns:xacro="http://www.ros.org/wiki/xacro">
-  <xacro:macro name="vehicle_system_multi_interface" params="name prefix serial_port state_update_frequency use_hardware world_frame_id body_frame_id map_frame_id">
+  <xacro:macro name="vehicle_system_multi_interface" params="name prefix serial_port state_update_frequency use_hardware world_frame_id body_frame_id map_frame_id use_pwm">
     <ros2_control name="${name}" type="system">
       <hardware>
@@ -10,4 +10,5 @@
           <param name="body_frame_id">${body_frame_id}</param>
           <param name="map_frame_id">${map_frame_id}</param>
+          <param name="use_pwm">${use_pwm}</param>
         </xacro:if>
         <xacro:unless value="${use_hardware}">

File: description/xacro/robot_system_multi_interface.urdf.xacro (robot description, xacro)
@@ -4,4 +4,5 @@
   <xacro:arg name="use_manipulator_hardware" default="false"/>
   <xacro:arg name="use_vehicle_hardware" default="false"/>
+  <xacro:arg name="use_pwm" default="true"/>
   <xacro:arg name="sim_robot_count" default="1"/>
   <xacro:arg name="serial_port" default="/dev/ttyUSB0"/>
@@ -16,4 +17,5 @@
   <xacro:property name="use_manipulator_hardware" value="$(arg use_manipulator_hardware)"/>
   <xacro:property name="use_vehicle_hardware" value="$(arg use_vehicle_hardware)"/>
+  <xacro:property name="use_pwm" value="$(arg use_pwm)"/>
   <xacro:property name="use_optitrack" value="$(arg use_optitrack)"/>
   <!-- Define constants -->
@@ -63,5 +65,6 @@
       world_frame_id="base_link"
       body_frame_id="${prefix}base_link"
-      map_frame_id="${prefix}map"/>
+      map_frame_id="${prefix}map"
+      use_pwm="${use_pwm}"/>
       <!-- Recursively call the macro for the next robot -->
       <xacro:instantiate_robots index="${index + 1}" count="${count}"/>
@@ -95,5 +98,6 @@
       world_frame_id="base_link"
       body_frame_id="${prefix}base_link"
-      map_frame_id="${prefix}map"/>
+      map_frame_id="${prefix}map"
+      use_pwm="${use_pwm}"/>
   </xacro:if>
 </robot>

Commit message: added same_initial_condition_startup_multirobot

File: description/ros2_control/vehicle_system_multi_interface.ros2_control.xacro (robot description, xacro)
@@ -1,5 +1,5 @@
 <?xml version="1.0"?>
 <robot xmlns:xacro="http://www.ros.org/wiki/xacro">
-  <xacro:macro name="vehicle_system_multi_interface" params="name prefix serial_port state_update_frequency use_hardware world_frame_id body_frame_id map_frame_id use_pwm">
+  <xacro:macro name="vehicle_system_multi_interface" params="name prefix serial_port state_update_frequency use_hardware world_frame_id body_frame_id map_frame_id same_initial_conditions use_pwm">
     <ros2_control name="${name}" type="system">
       <hardware>
@@ -10,4 +10,5 @@
           <param name="body_frame_id">${body_frame_id}</param>
           <param name="map_frame_id">${map_frame_id}</param>
+          <param name="same_initial_conditions">${same_initial_conditions}</param>
           <param name="use_pwm">${use_pwm}</param>
         </xacro:if>
@@ -18,4 +19,5 @@
           <param name="body_frame_id">${body_frame_id}</param>
           <param name="map_frame_id">${map_frame_id}</param>
+          <param name="same_initial_conditions">${same_initial_conditions}</param>
           <param name="use_pwm">${use_pwm}</param>
         </xacro:unless>

File: description/xacro/robot_system_multi_interface.urdf.xacro (robot description, xacro)
@@ -6,4 +6,5 @@
   <xacro:arg name="use_pwm" default="true"/>
   <xacro:arg name="sim_robot_count" default="1"/>
+  <xacro:arg name="same_initial_conditions" default="false"/>
   <xacro:arg name="serial_port" default="/dev/ttyUSB0"/>
   <xacro:arg name="state_update_frequency" default="250"/>
@@ -15,4 +16,5 @@
   <xacro:property name="description_package" value="$(arg description_package)"/>
   <xacro:property name="sim_robot_count" value="$(arg sim_robot_count)"/>
+  <xacro:property name="same_initial_conditions" value="$(arg same_initial_conditions)"/>
   <xacro:property name="serial_port" value="$(arg serial_port)"/>
   <xacro:property name="state_update_frequency" value="$(arg state_update_frequency)"/>
@@ -43,6 +45,7 @@
       <xacro:property name="circumference" value="${count * d_min}"/>
       <xacro:property name="radius" value="${circumference / (2 * pi)}"/>
-      <xacro:property name="x_pos" value="${radius * cos(angle)}"/>
-      <xacro:property name="y_pos" value="${radius * sin(angle)}"/>
+      <xacro:property name="x_pos" value="${0.0 if same_initial_conditions else radius * cos(angle)}"/>
+      <xacro:property name="y_pos" value="${0.0 if same_initial_conditions else radius * sin(angle)}"/>
+      <xacro:property name="yaw_pos" value="${0.0 if same_initial_conditions else angle}"/>
       <!-- Instantiate the robot -->
       <xacro:bluerov2_heavy_alpha_urdf
@@ -54,5 +57,5 @@
         rot_r="0.0"
         rot_p="0.0"
-        rot_y="${angle}"/>
+        rot_y="${yaw_pos}"/>
     <xacro:robot_system_multi_interface
       name="${prefix}ReachSystemMultiInterface"
@@ -70,4 +73,5 @@
       body_frame_id="${prefix}base_link"
       map_frame_id="${prefix}map"
+      same_initial_conditions="${same_initial_conditions}"
       use_pwm="${use_pwm}"/>
       <!-- Recursively call the macro for the next robot -->
@@ -104,4 +108,5 @@
       body_frame_id="${prefix}base_link"
       map_frame_id="${prefix}map"
+      same_initial_conditions="${same_initial_conditions}"
       use_pwm="${use_pwm}"/>
   </xacro:if>

Commit message: Refine camera launch and hardware behavior

File: description/ros2_control/vehicle_system_multi_interface.ros2_control.xacro (robot description, xacro)
@@ -1,5 +1,5 @@
 <?xml version="1.0"?>
 <robot xmlns:xacro="http://www.ros.org/wiki/xacro">
-  <xacro:macro name="vehicle_system_multi_interface" params="name prefix serial_port state_update_frequency use_hardware world_frame_id body_frame_id map_frame_id same_initial_conditions use_pwm">
+  <xacro:macro name="vehicle_system_multi_interface" params="name prefix serial_port state_update_frequency use_hardware world_frame_id body_frame_id map_frame_id same_initial_conditions use_pwm use_dvl dvl_host dvl_port">
     <ros2_control name="${name}" type="system">
       <hardware>
@@ -12,4 +12,7 @@
           <param name="same_initial_conditions">${same_initial_conditions}</param>
           <param name="use_pwm">${use_pwm}</param>
+          <param name="use_dvl">${use_dvl}</param>
+          <param name="dvl_host">${dvl_host}</param>
+          <param name="dvl_port">${dvl_port}</param>
         </xacro:if>
         <xacro:unless value="${use_hardware}">

File: description/xacro/robot_system_multi_interface.urdf.xacro (robot description, xacro)
@@ -11,4 +11,8 @@
   <xacro:arg name="description_package" default="ros2_control_blue_reach_5"/>
   <xacro:arg name="use_optitrack" default="false"/>
+  <xacro:arg name="world_frame" default="world"/>
+  <xacro:arg name="use_dvl" default="false"/>
+  <xacro:arg name="dvl_host" default="192.168.2.95"/>
+  <xacro:arg name="dvl_port" default="16171"/>
   <!-- <xacro:arg name="robot_name" default="bruce"/> -->
   <xacro:arg name="robot_name" default="dory"/>
@@ -23,4 +27,8 @@
   <xacro:property name="use_pwm" value="$(arg use_pwm)"/>
   <xacro:property name="use_optitrack" value="$(arg use_optitrack)"/>
+  <xacro:property name="world_frame" value="$(arg world_frame)"/>
+  <xacro:property name="use_dvl" value="$(arg use_dvl)"/>
+  <xacro:property name="dvl_host" value="$(arg dvl_host)"/>
+  <xacro:property name="dvl_port" value="$(arg dvl_port)"/>
   <xacro:property name="robot_name" value="$(arg robot_name)"/>
   <!-- Define constants -->
@@ -34,5 +42,5 @@
   <xacro:include filename="$(find ${description_package})/ros2_control/vehicle_system_multi_interface.ros2_control.xacro" />
   <!-- Instantiate the world -->
-  <xacro:sim_world/>
+  <xacro:sim_world world_frame="${world_frame}"/>
   <!-- Recursive Macro Definition -->
   <xacro:macro name="instantiate_robots" params="index count">
@@ -74,5 +82,8 @@
       map_frame_id="${prefix}map"
       same_initial_conditions="${same_initial_conditions}"
-      use_pwm="${use_pwm}"/>
+      use_pwm="${use_pwm}"
+      use_dvl="${use_dvl}"
+      dvl_host="${dvl_host}"
+      dvl_port="${dvl_port}"/>
       <!-- Recursively call the macro for the next robot -->
       <xacro:instantiate_robots index="${index + 1}" count="${count}"/>
@@ -109,5 +120,8 @@
       map_frame_id="${prefix}map"
       same_initial_conditions="${same_initial_conditions}"
-      use_pwm="${use_pwm}"/>
+      use_pwm="${use_pwm}"
+      use_dvl="${use_dvl}"
+      dvl_host="${dvl_host}"
+      dvl_port="${dvl_port}"/>
   </xacro:if>
 </robot>

File: description/xacro/world.xacro (robot description, xacro)
@@ -1,7 +1,7 @@
 <?xml version="1.0"?>
 <robot xmlns:xacro="http://ros.org/wiki/xacro">
-  <xacro:macro name="sim_world">
+  <xacro:macro name="sim_world" params="world_frame:=world">
       <!-- world origin -->
-    <link name="world">
+    <link name="${world_frame}">
         <visual>
         <origin rpy="0 0 0" xyz="0 0 0"/>
@@ -48,5 +48,5 @@
     <joint name="world_bottom_joint" type="fixed">
       <child link="world_bottom" />
-      <parent link="world" />
+      <parent link="${world_frame}" />
       <origin xyz="0.0 0.0 -8.0" rpy="0 0 0"/>
     </joint>
@@ -65,5 +65,5 @@
     <joint name="world_joint" type="fixed">
       <child link="base_link" />
-      <parent link="world" />
+      <parent link="${world_frame}" />
       <origin xyz="0.0 0.0 0.0" rpy="0 0 0"/>
     </joint>
